File: return_numpad/return_numpad.kicad_sch (KiCad schematic)
At the start: 34 parts, among them J1 Conn_01x04, SW1 SW_Push, SW10 SW_Push, SW11 SW_Push, SW12 SW_Push, SW13 SW_Push, SW14 SW_Push, SW15 SW_Push, SW16 SW_Push, SW2 SW_Push, SW3 SW_Push, SW4 SW_Push, SW5 SW_Push, SW6 SW_Push, SW7 SW_Push, SW8 SW_Push, SW9 SW_Push

Commit message: Finish main schematic, finish aux schematic, add production files.
Parts:
- removed D12: D_Small, Diode_THT:D_DO-35_SOD27_P7.62mm_Horizontal, symbol Device:D_Small
- removed SW12: SW_Push, Kailh_PG1353_Hotswap:Kailh-PG1353-Hotswap-1U, symbol Switch:SW_Push
- added C1: 1000uF, Resistor_THT:R_Axial_DIN0204_L3.6mm_D1.6mm_P2.54mm_Vertical, symbol Device:C_Small
- added D12, D21, D22, D23, D24, D25, D26, D27, D28, D29, D30, D31, D32, D33, D34, D35, D36: SK6812MINI, Keebio-Parts:SK6812-MINI-E, symbol LED:SK6812MINI
- added D17, D18, D19: D_Small, Diode_THT:D_DO-35_SOD27_P7.62mm_Horizontal, symbol Device:D_Small
- added R1: 500, Resistor_THT:R_Axial_DIN0207_L6.3mm_D2.5mm_P7.62mm_Horizontal, symbol Device:R_Small
- added SW17, SW19: SW_Push, Kailh_PG1353_Hotswap:Kailh-PG1353-Hotswap-1U, symbol Switch:SW_Push
- J1: footprint (none) -> Connector_PinHeader_2.54mm:PinHeader_1x04_P2.54mm_Vertical
Connections:
- net COL0: now also A1.10 (A5), SW17.1
- net COL1: now also A1.9 (A4)
- net COL2: now also A1.8 (A3), SW19.1
- net COL3: now also A1.7 (A2)
- net ROW0: now also A1.25 (D6)
- net ROW1: now also A1.24 (D5)
- net ROW2: now also A1.23 (D4)
- net ROW3: now also A1.22 (D3)
- net GND: now reaches J1.1 (Pin_1)
- net GND: now also A1.4 (GND), C1.2, D12.2 (VSS), D21.2 (VSS), D22.2 (VSS), D23.2 (VSS), D24.2 (VSS), D25.2 (VSS), D26.2 (VSS), D27.2 (VSS), D28.2 (VSS), D29.2 (VSS), D30.2 (VSS), D31.2 (VSS), D32.2 (VSS), D33.2 (VSS), D34.2 (VSS), D35.2 (VSS), D36.2 (VSS)
- net at J1.4 (Pin_4): now also D18.2 (A)
- net +3.3V: now reaches A1.2 (3V3)
- net +3.3V: now also C1.1, D12.4 (VDD), D18.1 (K), D21.4 (VDD), D22.4 (VDD), D23.4 (VDD), D24.4 (VDD), D25.4 (VDD), D26.4 (VDD), D27.4 (VDD), D28.4 (VDD), D29.4 (VDD), D30.4 (VDD), D31.4 (VDD), D32.4 (VDD), D33.4 (VDD), D34.4 (VDD), D35.4 (VDD), D36.4 (VDD)
- net ROW4: now reaches A1.21 (D2)
- net ROW4: now also D17.1 (K), D19.1 (K)
- net LED_DIN: now reaches A1.5 (A0)
- net LED_DIN: now also R1.1
- new net: D33.1 (DOUT), D34.3 (DIN)
- new net: D32.1 (DOUT), D33.3 (DIN)
- new net: D19.2 (A), SW19.2
- new net: D26.1 (DOUT), D27.3 (DIN)
- new net: D25.1 (DOUT), D26.3 (DIN)
- new net: D12.3 (DIN), D36.1 (DOUT)
- new net: D24.1 (DOUT), D25.3 (DIN)
- new net: D31.1 (DOUT), D32.3 (DIN)
- new net: D30.1 (DOUT), D31.3 (DIN)
- new net: D29.1 (DOUT), D30.3 (DIN)
- new net: D28.1 (DOUT), D29.3 (DIN)
- new net: D27.1 (DOUT), D28.3 (DIN)
- new net: D21.3 (DIN), R1.2
- new net: D23.1 (DOUT), D24.3 (DIN)
- new net: D22.1 (DOUT), D23.3 (DIN)
- new net: D17.2 (A), SW17.2
- new net: D21.1 (DOUT), D22.3 (DIN)
- new net: D35.1 (DOUT), D36.3 (DIN)
- new net: D34.1 (DOUT), D35.3 (DIN)
Other:
- moved on the sheet: J1
